File: yorp.kicad_sch (KiCad schematic)
At the start: 9 parts, among them J1 LT1085, U1 AP63203WU

Commit message: Add files via upload
Updated to 0.2
Parts:
- removed U1: AP63203WU, Package_TO_SOT_SMD:TSOT-23-6, symbol Regulator_Switching:AP63203WU
- added C6: 51pF, Capacitor_SMD:C_0805_2012Metric, symbol Device:C_Small
- added R1: 107K, Resistor_SMD:R_0805_2012Metric, symbol Device:R_Small
- added R2: 30.1K, Resistor_SMD:R_0805_2012Metric, symbol Device:R_Small
- added U2: AP63301WU-7, Package_TO_SOT_SMD:TSOT-23-6, symbol Regulator_Switching:AP63201WU
- L1: value 3.9u -> HPC 6045NC-4R7M
Connections:
- net 5V: now also U2.2 (EN), U2.3 (IN)
- net GND: now also R2.2, U2.4 (GND)
- net at C5.1, L1.1: now also U2.5 (SW)
- net at C5.2: now also U2.6 (BST)
- net 3.3V renamed 3.6V
- net 3.6V: now also C6.1, R1.1
- new net: C6.2, R1.2, R2.1, U2.1 (FB)
Other:
- note added: "3.6V BUCK CONVERTER"
- note removed: "3.3V BUCK CONVERTER"
- moved on the sheet: C1, C2, C3, C4
