File: yorp.kicad_pcb (KiCad board)
At the start: 4 copper layers, 22.8 x 12.2 mm, 10 parts, among them J1 LT1085, U1 AP63203WU

Commit message: Add files via upload
Updated to 0.2
Parts:
- removed U1: AP63203WU, Package_TO_SOT_SMD:TSOT-23-6
- added C6: 51pF, Capacitor_SMD:C_0805_2012Metric, F.Cu at (80.3, 82.2)
- added R1: 107K, Resistor_SMD:R_0805_2012Metric, F.Cu at (80.3, 80.2)
- added R2: 30.1K, Resistor_SMD:R_0805_2012Metric, F.Cu at (84.0, 80.2)
- added U2: AP63301WU, Package_TO_SOT_SMD:TSOT-23-6, F.Cu at (84.2, 83.6)
- L1: value 3.9u -> 4.7u
- moved G*** 5.83 mm to (88.8, 87.2)
- moved C7 2.38 mm to (79.7, 84.4)
- moved C5 0.36 mm to (87.6, 81.7)
- moved C1 0.12 mm to (79.1, 88.3)
- moved C2 0.12 mm to (81.5, 88.3)
- moved C3 0.10 mm to (83.8, 88.3)
- moved C4 0.10 mm to (86.1, 88.3)
- moved L1 0.10 mm to (92.3, 86.2)
Connections:
- net /3.3V renamed /3.6V
Routing:
- net /3.6V: track 23.6 -> 16.7 mm
- net /5V: track 9.70 -> 13.0 mm
- net GND: vias 45 -> 44
- added copper zone on F.Cu, net Net-(U2-FB)
Other:
- board size 22.8 x 12.2 mm -> 22.8 x 12.9 mm
- board text added: "IN"
- board text added: "OUT"
- board text added: "Yorp 0.2 AB 2025 MIT License"
- board text removed: "3.3V"
- board text removed: "5V"
- board text removed: "Yorp 0.1 AB 2025 MIT License"

Commit message: Add files via upload
Updated component values.
Parts:
- L1: value 4.7u -> HPC 6045NC-4R7M
- U2: value AP63301WU -> AP63301WU-7
Other:
- board text added: "6a0d230bddd8ba05 b44826ce3ea39b5a"
